File: video.kicad_sch (KiCad schematic)
At the start: 13 parts, among them J301 HDMI_C_1.3

Commit message: Cosmetics
Other:
- note added: "HDMI Type-C connector"
- moved on the sheet: C301, C302, C303, C304, C305, C306, C307, C308, C309, D301, J301, R301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

Commit message: First whole routing
Parts:
- J301: MFN C27636754 -> (none); MPN (none) -> C27636754
- R301, R302: MPN (none) -> C25744
Connections:
- net CONN_HDMI_D2-: now reaches C308.2, J301.3 (D2-)
- net CONN_HDMI_CLK+: now reaches C303.2, J301.11 (CK+)
- net CONN_HDMI_CLK-: now reaches C302.2, J301.12 (CK-)
- net HDMI_SCL: now reaches J301.15 (SCL), R301.2
- net HDMI_SDA: now reaches J301.16 (SDA), R302.2
- net CONN_HDMI_D2+: now reaches C309.2, J301.2 (D2+)
- net CONN_HDMI_D1+: now reaches C307.2, J301.5 (D1+)
- net CONN_HDMI_D1-: now reaches C306.2, J301.6 (D1-)
- net CONN_HDMI_D0+: now reaches C305.2, J301.8 (D0+)
- net CONN_HDMI_D0-: now reaches C304.2, J301.9 (D0-)
- net CK+ renamed HDMI_CK+
- net CK- renamed HDMI_CK-
- net D0+ renamed HDMI_D0+
- net D0- renamed HDMI_D0-
- net D1+ renamed HDMI_D1+
- net D1- renamed HDMI_D1-
- net D2+ renamed HDMI_D2+
- net D2- renamed HDMI_D2-
Other:
- moved on the sheet: C302, C303, C304, C305, C306, C307, C308, C309, R301, R302

Commit message: Update some component values and complete MPN for BOM
Parts:
- C301, C302, C303, C304, C305, C306, C307, C308, C309: value 100n -> 100nF; MPN (none) -> C190183
- D301: value NSR0530HT1G -> 1N5819WS; MPN (none) -> C191023
- J301: value HDMI_C_1.3 -> GT-HD005A-CGNG0
Changed lines of the file:
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@@
 			)
 		)
-		(property "Value" "NSR0530HT1G"
+		(property "Value" "1N5819WS"
 			(at 171.45 66.2939 90)
 			(effects
@@
 			)
 		)
+		(property "MPN" "C191023"
+			(at 168.91 64.77 0)
+			(effects
+				(font
+					(size 1.27 1.27)
+				)
+				(hide yes)
+			)
+		)
 		(pin "2"
 		)
@@
 			)
 		)
-		(property "Value" "100n"
+		(property "Value" "100nF"
 			(at 171.45 74.9362 0)
 			(effects
@@
 			)
 		)
+		(property "MPN" "C190183"
+			(at 168.91 73.66 0)
+			(effects
+				(font
+					(size 1.27 1.27)
+				)
+				(hide yes)
+			)
+		)
 		(pin "1"
 		)
@@
 			)
 		)
-		(property "Value" "100n"
+		(property "Value" "100nF"
 			(at 115.57 82.5562 0)
 			(effects
@@
 			)
 		)
+		(property "MPN" "C190183"
+			(at 113.03 81.28 0)
+			(effects
+				(font
+					(size 1.27 1.27)
+				)
+				(hide yes)
+			)
+		)
 		(pin "1"
 		)
@@
 			)
 		)
-		(property "Value" "HDMI_C_1.3"
+		(property "Value" "GT-HD005A-CGNG0"
 			(at 172.72 113.0299 0)
 			(effects
@@
 			)
 		)
-		(property "Value" "100n"
+		(property "Value" "100nF"
 			(at 87.63 82.5562 0)
 			(effects
@@
 			)
 		)
+		(property "MPN" "C190183"
+			(at 85.09 81.28 0)
+			(effects
+				(font
+					(size 1.27 1.27)
+				)
+				(hide yes)
+			)
+		)
 		(pin "1"
 		)
@@
 			)
 		)
-		(property "Value" "100n"
+		(property "Value" "100nF"
 			(at 124.46 82.5562 0)
 			(effects
@@
 		)
 		(property "Description" "Unpolarized capacitor, small symbol"
+			(at 121.92 81.28 0)
+			(effects
+				(font
+					(size 1.27 1.27)
+				)
+				(hide yes)
+			)
+		)
+		(property "MPN" "C190183"
 			(at 121.92 81.28 0)
 			(effects
@@
 			)
 		)
-		(property "Value" "100n"
+		(property "Value" "100nF"
 			(at 78.74 82.5562 0)
 			(effects
@@
 			)
 		)
+		(property "MPN" "C190183"
+			(at 76.2 81.28 0)
+			(effects
+				(font
+					(size 1.27 1.27)
+				)
+				(hide yes)
+			)
+		)
 		(pin "1"
 		)
@@
 			)
 		)
-		(property "Value" "100n"
+		(property "Value" "100nF"
 			(at 69.85 82.5562 0)
 			(effects
@@
 			)
 		)
+		(property "MPN" "C190183"
+			(at 67.31 81.28 0)
+			(effects
+				(font
+					(size 1.27 1.27)
+				)
+				(hide yes)
+			)
+		)
 		(pin "1"
 		)
@@
 			)
 		)
-		(property "Value" "100n"
+		(property "Value" "100nF"
 			(at 106.68 82.5562 0)
 			(effects
@@
 			)
 		)
+		(property "MPN" "C190183"
+			(at 104.14 81.28 0)
+			(effects
+				(font
+					(size 1.27 1.27)
+				)
+				(hide yes)
+			)
+		)
 		(pin "1"
 		)
@@
 			)
 		)
-		(property "Value" "100n"
+		(property "Value" "100nF"
 			(at 97.79 82.5562 0)
 			(effects
@@
 			)
 		)
+		(property "MPN" "C190183"
+			(at 95.25 81.28 0)
+			(effects
+				(font
+					(size 1.27 1.27)
+				)
+				(hide yes)
+			)
+		)
 		(pin "1"
 		)
@@
 			)
 		)
-		(property "Value" "100n"
+		(property "Value" "100nF"
 			(at 60.96 82.5562 0)
 			(effects
@@
 			(at 58.42 81.28 0)
 			(effects
+				(font
+					(size 1.27 1.27)
+				)
+				(hide yes)
+			)
+		)
+		(property "MPN" "C190183"
+			(at 58.42 81.28 0)
+			(effects
