File: ram.kicad_sch (KiCad schematic)
At the start: 8 parts, among them U501 MT48LC16M16A2

Commit message: First whole routing
Parts:
- removed C505, C506, C507: 100n, Capacitor_SMD:C_0201_0603Metric, symbol Device:C_Small
- removed U501: MT48LC16M16A2, Package_BGA_Extra:Micron_VFBGA-64_8.0x8.0mm_Layout9x9_P0.8mm, symbol Memory_RAM_Extra:MT48LC16M16A2
- added U2: ~, Package_BGA_Extra:FBGA-25_8x6mm_Layout5x5_P1mm, symbol Memory_RAM_Extra:S80KS2562
- C501, C502, C503: footprint Capacitor_SMD:C_0201_0603Metric -> Capacitor_SMD:C_0402_1005Metric
- C504: value 100n -> 10u; footprint Capacitor_SMD:C_0201_0603Metric -> Capacitor_SMD:C_0402_1005Metric
Connections:
- net DQ0: now also U2.D3 (DQ0)
- net DQ1: now also U2.D2 (DQ1)
- net DQ2: now also U2.C4 (DQ2)
- net DQ3: now also U2.D4 (DQ3)
- net DQ4: now also U2.D5 (DQ4)
- net DQ5: now also U2.E3 (DQ5)
- net DQ6: now also U2.E2 (DQ6)
- net DQ7: now also U2.E1 (DQ7)
- net GND: now also U2.B3 (VSS), U2.C1 (VSSQ), U2.E5 (VSSQ)
- net +3V3 renamed +1V8
- net +1V8: now also U2.B4 (VCC), U2.D1 (VCCQ), U2.E4 (VCCQ)
- new net: U2.A2 (RFU), U2.A5 (RFU), U2.B5 (RFU), U2.C2 (RFU), U2.C5 (RFU)
- new net CK_N: U2.B1 (CK#)
- new net CK_P: U2.B2 (CK)
- new net CS#: U2.A3 (CS#)
- new net RESET#: U2.A4 (RESET#)
- new net RWDS: U2.C3 (RWDS)
Other:
- note added: "HyperRAM(TM) (256Mb)"
- note removed: "SDR SDRAM (256Mb)"
- moved on the sheet: C501, C502, C503

Commit message: Update some component values and complete MPN for BOM
Parts:
- C501, C502, C503: value 100n -> 100nF; MPN (none) -> C1525
- C504: value 10u -> 10uF; MPN (none) -> C15525
- U2: value ~ -> W958D8NBYA5I; MPN (none) -> C7420405
Changed lines of the file:
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@@
 			)
 		)
-		(property "Value" "100n"
+		(property "Value" "100nF"
 			(at 124.46 58.4262 0)
 			(effects
@@
 		)
 		(property "Description" "Unpolarized capacitor, small symbol"
+			(at 121.92 57.15 0)
+			(effects
+				(font
+					(size 1.27 1.27)
+				)
+				(hide yes)
+			)
+		)
+		(property "MPN" "C1525"
 			(at 121.92 57.15 0)
 			(effects
@@
 			)
 		)
-		(property "Value" "~"
+		(property "Value" "W958D8NBYA5I"
 			(at 150.7841 66.04 0)
 			(effects
@@
 		)
 		(property "Description" ""
+			(at 146.05 81.28 0)
+			(effects
+				(font
+					(size 1.27 1.27)
+				)
+				(hide yes)
+			)
+		)
+		(property "MPN" " C7420405 "
 			(at 146.05 81.28 0)
 			(effects
@@
 			)
 		)
-		(property "Value" "10u"
+		(property "Value" "10uF"
 			(at 106.68 58.4262 0)
 			(effects
@@
 		)
 		(property "Description" "Unpolarized capacitor, small symbol"
+			(at 104.14 57.15 0)
+			(effects
+				(font
+					(size 1.27 1.27)
+				)
+				(hide yes)
+			)
+		)
+		(property "MPN" "C15525"
 			(at 104.14 57.15 0)
 			(effects
@@
 			)
 		)
-		(property "Value" "100n"
+		(property "Value" "100nF"
 			(at 115.57 58.4262 0)
 			(effects
@@
 		)
 		(property "Description" "Unpolarized capacitor, small symbol"
+			(at 113.03 57.15 0)
+			(effects
+				(font
+					(size 1.27 1.27)
+				)
+				(hide yes)
+			)
+		)
+		(property "MPN" "C1525"
 			(at 113.03 57.15 0)
 			(effects
@@
 			)
 		)
-		(property "Value" "100n"
+		(property "Value" "100nF"
 			(at 133.35 58.4262 0)
 			(effects
@@
 			(at 130.81 57.15 0)
 			(effects
+				(font
+					(size 1.27 1.27)
+				)
+				(hide yes)
+			)
+		)
+		(property "MPN" "C1525"
+			(at 130.81 57.15 0)
+			(effects

Commit message: Last minute changes before sending to JLCPCB
Parts:
- U2: footprint Package_BGA_Extra:FBGA-25_8x6mm_Layout5x5_P1mm -> Package_BGA_Extra:FBGA-25_8x6mm_Layout5x6_P1mm
Changed lines of the file:
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@@
 			)
 		)
-		(property "Footprint" "Package_BGA_Extra:FBGA-25_8x6mm_Layout5x5_P1mm"
+		(property "Footprint" "Package_BGA_Extra:FBGA-25_8x6mm_Layout5x6_P1mm"
 			(at 146.812 103.124 0)
 			(effects
